Commit message: DHBW elements and conveyor belt in URDF

File: iwtros_description/urdf/conveyor/conveyor.urdf.xacro (robot description, xacro)
@@ -18,8 +18,8 @@
         <origin rpy="0 0 0" xyz="0 0 0"/>
         <geometry>
-          <mesh filename="package://robots_ee_pkg/meshes/conveyor/visual/bandumlaufsystem.dae" scale="0.001 0.001 0.001"/>
+          <mesh filename="package://iwtros_description/meshes/conveyor/visual/bandumlaufsystem.dae" scale="0.001 0.001 0.001"/>
         </geometry>
-        <material name="grey">
-          <color rgba="0.5 0.5 0.5 1"/>
+        <material name="darkgray">
+          <color rgba="0.3 0.3 0.3 1.0"/>
         </material>
       </visual>
@@ -27,5 +27,5 @@
         <origin rpy="0 0 0" xyz="0 0 0"/>
           <geometry>
-            <mesh filename="package://robots_ee_pkg/meshes/conveyor/collision/bandumlaufsystem.stl" scale="0.001 0.001 0.001" />
+            <mesh filename="package://iwtros_description/meshes/conveyor/collision/bandumlaufsystem.stl" scale="0.001 0.001 0.001" />
           </geometry>
       </collision>
@@ -37,4 +37,31 @@
       <mu2>0.4</mu2>
     </gazebo>
+    <link name="display">
+      <inertial>
+        <mass value="100"/>
+        <origin xyz="0 0 0" />
+        <inertia  ixx="1" ixy="0.0"  ixz="0.0"  iyy="1"  iyz="0.0"  izz="1" />
+      </inertial>
+      <visual>
+        <origin rpy="0 0 0" xyz="0 0 0"/>
+        <geometry>
+          <box size="0.3 0.01 0.5"/>
+        </geometry>
+        <material name="white">
+          <color rgba="1.0 1.0 1.0 1.0"/>
+        </material>
+      </visual>
+      <collision>
+        <origin rpy="0 0 0" xyz="0 0 0"/>
+          <geometry>
+            <box size="0.3 0.01 0.5"/>
+          </geometry>
+      </collision>
+    </link>
+    <joint name="${parent}_display_joint" type="fixed">
+        <parent link="${parent}"/>
+        <child link="display"/>
+        <origin xyz="0 -0.6 1.25"/>
+    </joint>
   </xacro:macro>
 </robot>

File: iwtros_description/urdf/kuka_robot/iiwa7.urdf.xacro (robot description, xacro)
@@ -6,5 +6,5 @@
   <xacro:arg name="robot_name" default="iiwa"/>
   <xacro:arg name="robot_param" default="/iiwa/iiwa_description"/>
-  <xacro:arg name="workcell_parent" default="world_interface"/>
+  <xacro:arg name="workcell_parent" default="world"/>
   <link name="$(arg workcell_parent)"/>
   <!-- origin is given as in the iwt_envirnment.xacro for urdf
@@ -12,8 +12,15 @@
   <xacro:include filename="$(find iwtros_description)/urdf/kuka_robot/kuka_iiwa7.urdf.xacro" />
   <xacro:kuka_iiwa7_table_urdf table_prefix="$(arg robot_name)" table_parent="$(arg workcell_parent)">
-    <origin xyz="0 0 0" rpy="0 0 0" />
+    <origin xyz="0 0 1" rpy="0 0 0" />
   </xacro:kuka_iiwa7_table_urdf>
   <gazebo reference="$(arg workcell_parent)">
       <gravity>true</gravity>
   </gazebo>
+  <!-- ToDo: Missing Gazebo plugins-->
+  <xacro:include filename="$(find iwtros_description)/urdf/conveyor/dhbw.xacro" />
+  <xacro:dhbw_system parent="$(arg workcell_parent)" />
+  <xacro:include filename="$(find iwtros_description)/urdf/conveyor/conveyor.urdf.xacro" />
+   <xacro:conveyor_system parent="$(arg workcell_parent)">
+    <origin xyz="-1 -5.5 1" rpy="0 0 1.57" />
+  </xacro:conveyor_system>
 </robot>

File: iwtros_description/urdf/kuka_robot/kuka_iiwa7.urdf.xacro (robot description, xacro)
@@ -7,5 +7,5 @@
   <xacro:include filename="$(find iiwa_description)/urdf/materials.xacro" />
   <!--Import the lbr iiwa macro -->
-  <xacro:include filename="$(find iiwa_description)/urdf/kuka_iiwa7.xacro"/>
+  <xacro:include filename="$(find iiwa_description)/urdf/iiwa7.xacro"/>
   <xacro:include filename="$(find wsg_50_simulation)/urdf/wsg_50.urdf.xacro" />
   <xacro:include filename="$(find iwtros_description)/urdf/table/add_table.urdf.xacro" />

File: iwtros_description/urdf/table/add_table.urdf.xacro (robot description, xacro)
@@ -22,5 +22,5 @@
         <origin xyz="0 0 -${0.53}" rpy="${PI/2} 0 -${PI/2}"/>
         <geometry>
-          <mesh filename="package://robots_ee_pkg/meshes/lf044_rough.dae" scale="0.001 0.001 0.001"/>
+          <mesh filename="package://iwtros_description/meshes/lf044_rough.dae" scale="0.001 0.001 0.001"/>
         </geometry>
         <material name="grey">
@@ -31,5 +31,5 @@
         <origin xyz="0 0 -${0.53}" rpy="${PI/2} 0 -${PI/2}"/>
           <geometry>
-            <mesh filename="package://robots_ee_pkg/meshes/lf044_rough.stl" scale="0.001 0.001 0.001"/>
+            <mesh filename="package://iwtros_description/meshes/lf044_rough.stl" scale="0.001 0.001 0.001"/>
           </geometry>
       </collision>

Commit message: Element position correction

File: iwtros_description/urdf/conveyor/conveyor.urdf.xacro (robot description, xacro)
@@ -46,5 +46,5 @@
         <origin rpy="0 0 0" xyz="0 0 0"/>
         <geometry>
-          <box size="0.3 0.01 0.5"/>
+          <box size="0.55 0.01 0.67"/>
         </geometry>
         <material name="white">
@@ -55,5 +55,5 @@
         <origin rpy="0 0 0" xyz="0 0 0"/>
           <geometry>
-            <box size="0.3 0.01 0.5"/>
+            <box size="0.55 0.01 0.67"/>
           </geometry>
       </collision>
@@ -62,5 +62,5 @@
         <parent link="${parent}"/>
         <child link="display"/>
-        <origin xyz="0 -0.6 1.25"/>
+        <origin xyz="0 -0.6 1.335"/>
     </joint>
   </xacro:macro>

File: iwtros_description/urdf/conveyor/dhbw.xacro (robot description, xacro)
@@ -38,5 +38,5 @@
         <origin rpy="0 0 0" xyz="0 0 0"/>
         <geometry>
-          <box size="0.8 0.3 0.81"/>
+          <box size="0.46 0.24 0.81"/>
         </geometry>
         <material name="green">
@@ -47,5 +47,5 @@
         <origin rpy="0 0 0" xyz="0 0 0"/>
           <geometry>
-            <box size="0.8 0.3 0.81"/>
+            <box size="0.46 0.24 0.81"/>
           </geometry>
       </collision>
@@ -54,5 +54,5 @@
         <parent link="${parent}"/>
         <child link="dbhwconveyor"/>
-        <origin xyz="0 0.76 0.405"/>
+        <origin xyz="0.53 0.67 0.405"/>
     </joint>
     <link name="sensor">
@@ -65,5 +65,5 @@
         <origin rpy="0 0 0" xyz="0 0 0"/>
         <geometry>
-          <box size="0.2 0.15 0.2"/>
+          <box size="0.15 0.15 0.3"/>
         </geometry>
         <material name="yellow">
@@ -74,5 +74,5 @@
         <origin rpy="0 0 0" xyz="0 0 0"/>
           <geometry>
-            <box size="0.2 0.15 0.2"/>
+            <box size="0.15 0.15 0.3"/>
           </geometry>
       </collision>
@@ -81,5 +81,5 @@
         <parent link="${parent}"/>
         <child link="sensor"/>
-        <origin xyz="0 3 0"/>
+        <origin xyz="0.205 0.745 1.15"/>
     </joint>
   </xacro:macro>
