Commit message: KUKA table change position in x axis

File: iwtros_description/urdf/conveyor/dhbw.xacro (robot description, xacro)
@@ -54,5 +54,5 @@
         <parent link="${parent}"/>
         <child link="dbhwconveyor"/>
-        <origin xyz="0.53 0.67 0.405"/>
+        <origin xyz="0.44 0.67 0.405"/>   <!--Moved the KUKA Table arount 0.091 m-->
     </joint>
     <link name="sensor">
@@ -81,5 +81,5 @@
         <parent link="${parent}"/>
         <child link="sensor"/>
-        <origin xyz="0.205 0.745 1.15"/>
+        <origin xyz="0.14 0.745 1.15"/>  <!--Moved the KUKA Table arount 0.091 m-->
     </joint>
   </xacro:macro>
