Commit message: Simulation update

File: iwtros_description/urdf/kuka_robot/kuka_iiwa7.gazebo.xacro (robot description, xacro)
@@ -33,5 +33,5 @@
     </gazebo>
     <gazebo reference="${robot_name}_link_4">
-      <turnGravityOff>true</turnGravityOff>
+      <turnGravityOff>true</turnGravityOff>MYROBOT
       <selfCollide>true</selfCollide>
       <material>Gazebo/Orange</material>
@@ -39,10 +39,5 @@
       <mu2>0.2</mu2>
     </gazebo>
-    <gazebo reference="${robot_name}_link_5">
-      <turnGravityOff>true</turnGravityOff>
-      <selfCollide>true</selfCollide>
-      <material>Gazebo/Orange</material>
-      <mu1>0.2</mu1>
-      <mu2>0.2</mu2>
+    <gazebo reference="${robot_name}_link_5">MYROBOT
     </gazebo>
     <gazebo reference="${robot_name}_link_6">
@@ -62,5 +57,6 @@
     <gazebo>
       <plugin name="gazebo_ros_control" filename="libgazebo_ros_control.so">
-        <robotParam>${robot_parameter_name}</robotParam>
+        <robotNamespace>/{robot_name}</robotNamespace>
+        <robotSimType>gazebo_ros_control/DefaultRobotHWSim</robotSimType>
         <legacyModeNS>false</legacyModeNS>
       </plugin>
